File: Hardware/24V_SSTC/SSTC.sch (EAGLE design)
At the start: 40 parts, among them IC1 NE555, J5 PIN1-2, Q1 IRF512, Q2 IRF512, Q3 BUZ11BH, Q4 BUZ11BH, T1 BD242C, T2 BD242C

Commit message: Fertigstellung der SSTC Kleinere Bugfixes im UI
Parts:
- removed J1: (no value), con-jack:DCJ0303
- removed J5: PIN1-2, con-faston:PIN1-2
- added C1, C5, C6, C7: 100n, rcl:C-EU075-032X103
- added C10: (no value), rcl:C-EU102_152-062X184
- added C11: (no value), rcl:CPOL-EUE7.5-18
- added C8: 1m, rcl:CPOL-EUE5-10.5
- added C9: 22µ, rcl:CPOL-EUE5-8.5
- added P1: (no value), pot:3RP/1610N
- added R11: 168k, rcl:R-EU_0309/12
- added R12: 22k, rcl:R-EU_0309/12
- added R3: 80k, rcl:R-EU_0207/10
- added R6: 168k, rcl:R-EU_0207/10
- added R7: 22k, rcl:R-EU_0207/10
- added U$3: T50_INDUCTOR, toroid:T50_INDUCTOR
- added X2: (no value), con-wago-500:W237-102
- added X3: (no value), con-wago-500:W237-112
- D1, D2: device diode:DIODE-DO41-7.6 -> diode:DIODE-DO35-10
- D10, D11, D12, D8, D9: device diode:DIODE-MELF-MLL41 -> diode:DIODE-D-10
- D3, D4, D5, D6, D7: device diode:SCHOTTKY-DIODESMD -> diode:SCHOTTKY-DIODEF126Z12
- R1, R10, R4, R5: device rcl:R-EU_R2512 -> rcl:R-EU_0207/10
- R2: value (none) -> 38k; device pot:3RP/1610N -> rcl:R-EU_0207/10
- R8: device rcl:R-EU_R2512 -> rcl:R-EU_0309/12
- R9: device rcl:R-EU_0309/12 -> rcl:R-EU_0613/5V
- Z1, Z2: device diode:ZENER-DIODESOD80C -> diode:ZENER-DIODEDO35Z10
Connections:
- new net N$16: C9.+, Q4.G, R10.1, T2.B, Z2.C
- new net N$17: R8.1, T2.E
- new net N$18: IC1.DIS, R5.1, R6.1
- new net N$19: C5.1, IC1.TRE, IC1.TRI, R5.2
- new net N$20: P1.S, R6.2
- new net N$21: P1.A, R11.2
- new net N$22: Q3.G, R12.1, S1.P
- new net N$23: IC1.OUT, S1.S
- new net N$24: S1.O, U$2.P$1
- new net VCC/2: C6.1, C8.+, D7.C, IC1./RES, IC1.VCC+, P1.E, Q4.S, R12.2, R3.2, R7.2, R8.2
- net GND: now also C1.2, C10.1, C11.-, C5.2, C6.2, C7.2, C8.-, C9.-, IC1.GND, Q3.S, R11.1, R2.1, T2.C, U$2.P$2, U$3.CA, X2-1.KL, Z2.A; no longer J1.1
- net N$10: now also D7.A, Q3.D, R7.1
- net N$11: now also C7.1, D2.C
- net N$13: now also C10.2, U$3.CB
- net N$14: now also X3.KL; no longer J5.1
- net N$15: now also X2-2.KL; no longer J1.2, J1.3
- net N$5: now also C1.1
- net N$6: now also R2.2, R3.1, U$1.C1B; no longer U$1.C1A
- net N$7: now also U$1.C1A; no longer U$1.C1B
- net VCC: now also C11.+, Q4.D, R10.2
Other:
- moved on the sheet: D7, IC1, KK1, Q2, Q3, Q4, R10, R5, R8, R9, S1, T2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
