File: Hardware/Netzteil/Netzteil_V_1.0.sch (EAGLE design)
At the start: 29 parts, among them IC1 7812L, IC3 LM2574HVN-5.0, IC4 LM2574HVN-3.3, X1 87758-1016

Commit message: Letzte Änderungen an Netzteil, OP und IP Board
Connections:
- net N$15 renamed -12V
- net N$17 renamed +12V
- net N$19 renamed 3V3
- net N$22 renamed 5V
