File: Hardware/Mainboard/Mainboard.brd (EAGLE design)
At the start: 130 x 100 mm, 86 parts, among them IC1 24AA256SN, IC3 ATMEGA2560-16AU, Q1 12.288Mhz, Q6 BSS123, Q7 BSS123, Q8 BSS123, Q9 BSS123, T1 FZT751TA, X8 MAB5SH, Y1 CSTCE16M0V53-R0 16MHZ

Commit message: Minor Board Fixes
Parts:
- removed D3: CD1206-S01575, diode:MINIMELF
- added D2: 1n4148, diode:SOD-123_MINI-SMA
- D1: value 1N4148DO35-10 -> 1N4148; device diode:DO35-10 -> diode:SOD-123_MINI-SMA
- R12: device rcl:0207/10 -> rcl:R0805
- moved D1 3.81 mm to (94.0, 22.9)
- moved R12 2.54 mm to (94.0, 20.3)
- moved Q1 1.27 mm to (73.7, 67.3)
Connections:
- net +5V: now also D2.C; no longer D3.C
- net PB0: no longer SD_SOCKET.8
- net PH6: now also SD_SOCKET.8
- net RESET: now also D2.A; no longer D3.A
Routing:
- net PH6: track 0.00 -> 56.7 mm
- net N$13: track 6.66 -> 15.4 mm
- net N$15: track 7.62 -> 10.7 mm
- net PB0: track 58.4 -> 55.9 mm
- net N$7: track 23.5 -> 22.2 mm
- net N$6: track 10.1 -> 8.86 mm
- net RESET: track 74.3 -> 73.6 mm
Other:
- board text added: "Teslacontroller Mainboard by Michael Loose@FHWS Rev 1.0 05/19"
- board text removed: "Teslacontroller Mainboard by Michael Loose FHWS 05/19"
