File: Hardware/Mainboard/Mainboard.brd (EAGLE design)
At the start: 130 x 100 mm, 86 parts, among them IC1 24AA256SN, IC3 ATMEGA2560-16AU, Q1 12.288Mhz, Q6 BSS123, Q7 BSS123, Q8 BSS123, Q9 BSS123, T1 FZT751TA, X8 MAB5SH, Y1 CSTCE16M0V53-R0 16MHZ

Commit message: minor fixes
Parts:
- turned D1 to 180 degrees
Connections:
- net N$15: now also D1.C; no longer D1.A
- net N$16: now also D1.A; no longer D1.C
Routing:
- net PE: track 5.08 -> 0.00 mm
Changed lines of the file:
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@@
 <attribute name="VALUE" x="57.785" y="24.13" size="1.27" layer="27" rot="R90"/>
 </element>
-<element name="D1" library="diode" library_urn="urn:adsk.eagle:library:210" package="SOD-123_MINI-SMA" package3d_urn="urn:adsk.eagle:package:43457/2" value="1N4148" x="93.98" y="22.86">
-<attribute name="NAME" x="90.932" y="24.003" size="1.27" layer="25"/>
-<attribute name="VALUE" x="90.932" y="20.447" size="1.27" layer="27"/>
+<element name="D1" library="diode" library_urn="urn:adsk.eagle:library:210" package="SOD-123_MINI-SMA" package3d_urn="urn:adsk.eagle:package:43457/2" value="1N4148" x="93.98" y="22.86" rot="R180">
+<attribute name="NAME" x="97.028" y="21.717" size="1.27" layer="25" rot="R180"/>
+<attribute name="VALUE" x="97.028" y="25.273" size="1.27" layer="27" rot="R180"/>
 </element>
 <element name="D2" library="diode" library_urn="urn:adsk.eagle:library:210" package="SOD-123_MINI-SMA" package3d_urn="urn:adsk.eagle:package:43457/2" value="1n4148" x="43.18" y="5.08">
@@
 <contactref element="X8" pad="PE"/>
 <contactref element="X8" pad="PE@"/>
-<wire x1="91.44" y1="2.54" x2="96.52" y2="2.54" width="0.508" layer="1"/>
+<wire x1="91.44" y1="2.54" x2="96.52" y2="2.54" width="0" layer="19" extent="1-1"/>
 </signal>
 <signal name="GND">
@@
 <contactref element="X8" pad="4"/>
 <contactref element="R12" pad="1"/>
-<contactref element="D1" pad="A"/>
 <wire x1="99.06" y1="15.24" x2="99.06" y2="16.19" width="0.508" layer="1"/>
 <wire x1="99.06" y1="15.24" x2="99.06" y2="16.51" width="0.508" layer="1"/>
 <wire x1="99.06" y1="16.51" x2="95.25" y2="20.32" width="0.508" layer="1"/>
-<wire x1="95.78" y1="22.86" x2="95.78" y2="20.85" width="0.508" layer="1"/>
-<wire x1="95.78" y1="20.85" x2="95.25" y2="20.32" width="0.508" layer="1"/>
 <wire x1="94.93" y1="20.32" x2="95.25" y2="20.32" width="0.508" layer="1"/>
+<contactref element="D1" pad="C"/>
+<wire x1="94.93" y1="20.32" x2="95.78" y2="21.17" width="0.508" layer="1"/>
+<wire x1="95.78" y1="21.17" x2="95.78" y2="22.86" width="0.508" layer="1"/>
 </signal>
 <signal name="N$16">
 <contactref element="OK1" pad="3"/>
 <contactref element="X8" pad="5"/>
-<contactref element="D1" pad="C"/>
 <wire x1="88.9" y1="15.24" x2="88.9" y2="19.58" width="0.508" layer="1"/>
+<contactref element="D1" pad="A"/>
+<wire x1="92.445" y1="23.125" x2="92.18" y2="22.86" width="0.508" layer="1"/>
 <wire x1="88.9" y1="19.58" x2="92.18" y2="22.86" width="0.508" layer="1"/>
-<wire x1="92.18" y1="22.86" x2="95.25" y2="25.93" width="0.254" layer="1"/>
-<wire x1="95.25" y1="25.93" x2="95.25" y2="27.94" width="0.254" layer="1"/>
+<wire x1="95.25" y1="27.94" x2="95.25" y2="25.93" width="0.254" layer="1"/>
+<wire x1="95.25" y1="25.93" x2="92.18" y2="22.86" width="0.254" layer="1"/>
 </signal>
 <signal name="N$17">
