File: Hardware/Mainboard/Mainboard.sch (EAGLE design)
At the start: 86 parts, among them IC1 24AA256SN, IC3 ATMEGA2560-16AU, Q1 12.288Mhz, Q6 BSS123, Q7 BSS123, Q8 BSS123, Q9 BSS123, T1 FZT751TA, X8 MAB5SH, Y1 CSTCE16M0V53-R0 16MHZ

Commit message: Minor Board Fixes
Parts:
- removed D3: CD1206-S01575, diode:DIODE-MINIMELF
- added D2: 1n4148, diode:CGRM4001-G
- D1: value 1N4148DO35-10 -> 1N4148; device diode:1N4148DO35-10 -> diode:CGRM4001-G
- R12: device rcl:R-EU_0207/10 -> rcl:R-EU_R0805
Connections:
- net +5V: now also D2.C; no longer D3.C
- net PB0: no longer SD_SOCKET.8
- net PH6: now also SD_SOCKET.8
- net RESET: now also D2.A; no longer D3.A
